File: src/hardware/NodeNetSoh_motherboard_V0.1/NodeNetSoh_motherboard_V0.1.kicad_sch (KiCad schematic)
At the start: 0 parts

Commit message: feat: update firmware blink flow, wb timer, and hardware/docs
Parts:
- added J1: RJHSE538102, MyLibrary:AMPHENOL_RJHSE538102, symbol MyLibrary_sym:RJHSE538102
Other:
- added sheet ColorLight i9 (ColorLight i9.kicad_sch)
- added sheet POWER Module (Modules/NodeNet_PWR_Module/NodeNet_PWR_Module.kicad_sch)
- added sheet modbus0 (rs485Module.kicad_sch)
- added sheet modbus1 (rs485Module.kicad_sch)
- added sheet modbus2 (rs485Module.kicad_sch)
- added sheet modbus3 (rs485Module.kicad_sch)
- added sheet nodeNet module (rs485Module.kicad_sch)
